Commit message: feat: Agent.joint_tolerance, per-joint tolerance, tolerance write-back, docs update
Joint tolerance system:
- Agent.joint_tolerance property with fallback chain (Action > Agent > default 0.01)
- JointAction tolerance write-back: resolved once at first execute() and written to action.tolerance
- Per-joint tolerance via dict keyed by joint name (e.g. rail_joint: 0.005)
- _resolve_joint_tolerance() handles None/scalar/dict/list with consistent default fallback
- List out-of-range fallback changed from clamp-to-last to _DEFAULT_JOINT_TOLERANCE

Prismatic support improvements:
- Per-joint-type kinematic fallback velocity (revolute: 2.0 rad/s, prismatic: 0.5 m/s)
- rail_arm_robot.urdf improvements
- rail_arm_demo.py with per-joint tolerance example

Test improvements:
- TestResolveJointTolerance: all-index loops, merged dict tests, list fallback to default
- TestAgentJointToleranceIntegration: tolerance write-back, explicit override, setter
- TestRailArmIK: 6 IK tests with reachability checks
- Fixture consolidation (pybullet_env, arm_sim in conftest.py)
- Duplicate test removal, run_arm_until_idle simplification

Documentation:
- Tutorial 4 (arm-pick-drop): JointAction tolerance reference (scalar/dict/agent fallback/write-back)
- Tutorial 5 (arm-ee-control): prismatic joints & rail arm section, rail_arm_demo link
- Architecture overview: tolerance resolution, prismatic fallback velocity, joint_tolerance
- examples/index.md, quickstart.md: rail_arm_demo, EE demos added
- CHANGELOG: linear joint entries
- Design spec: Draft -> Implemented

File: robots/rail_arm_robot.urdf (robot description, URDF)
Before this commit: robot rail_arm_robot, 6 links, 5 joints
Links:
- link rail_platform_link: geometry collision cylinder length=0.05 radius=0.05; visual cylinder length=0.05 radius=0.05
- link world_link: geometry collision box size=0.08 0.08 1.2; visual box size=0.08 0.08 1.0
Joints:
- joint base_to_shoulder: origin xyz=0.0 0.0 0.05 rpy=0 0 0 -> xyz=0.1 0.0 0.05 rpy=0 0 0
