Commit message: feat: kinematic mobile manipulator with IK, drop_relative_pose, and test improvements
- Rewrite mobile_manipulator_demo.py for kinematic mode
- Add IK support: auto-detect movable joints, lock continuous wheels
- Add ik_joint_names parameter for explicit joint specification
- Add drop_relative_pose to DropAction for relative drop positioning
- Fix attachment tracking, base movement lag, drop pose alignment
- Replace magic number JOINT_FIXED=4 with p.JOINT_FIXED
- Tighten test assertions (0.3 -> COARSE_TOL), remove dead code
- Fix wheel lock tests to use non-zero initial positions
- Deduplicate TestIKJointNames (8 -> 4 tests, remove auto-mode dupes)
- Add design docs for kinematic mobile manipulator spec

File: robots/mobile_manipulator.urdf (robot description, URDF)
Before this commit: robot mobile_manipulator, 8 links, 7 joints
Joints:
- joint base_to_mount: origin xyz=-0.1 0.0 0.15 rpy=0 0 0 -> xyz=0.25 0.0 0.15 rpy=0 0 0
