Commit message: feat: add EventBus, SDF loader, and resolve_model rename
EventBus — lightweight pub/sub for simulation lifecycle events:
- SimEvents constants (PRE_STEP, POST_STEP, OBJECT_SPAWNED, AGENT_SPAWNED,
  COLLISION_STARTED/ENDED, ACTION_STARTED/COMPLETED, PRE_UPDATE, POST_UPDATE)
- Global bus (sim.events) and per-entity bus (agent.events)
- Priority ordering, exception isolation, handler management
- event_bus_demo.py example covering all event types

SDF loader — bulk-load SDF files as SimObjects:
- SimObject.from_sdf() wraps p.loadSDF() with batch_spawn() for GUI speedup
- world_loader.py: load_mesh_directory() for bulk OBJ/STL loading
  (load_rmf_world kept as backward-compatible alias)
- warehouse_layout.sdf: self-contained multi-model demo (ground + 4 shelves)
- sdf_demo.py example demonstrating multi-model, scaling, and mesh directory

resolve_urdf → resolve_model rename:
- resolve_model() handles both URDF and SDF; resolve_urdf() kept as alias
- Updated all examples, docs, README, CHANGELOG references

Other improvements:
- Added <inertial> to mobile_robot, arm_robot, rail_arm_robot URDFs
- 49 test files, comprehensive coverage for events + SDF + world_loader

File: robots/arm_robot.urdf (robot description, URDF)
Before this commit: robot articulated_arm_robot, 5 links, 4 joints
Links:
- link base_link: mass None -> 2.0
- link elbow_link: mass None -> 0.3
- link end_effector: mass None -> 0.1
- link shoulder_link: mass None -> 0.5
- link wrist_link: mass None -> 0.2

File: robots/mobile_robot.urdf (robot description, URDF)
Before this commit: robot mobile_robot, 5 links, 4 joints
Links:
- link base_link: mass None -> 10.0
- link camera: mass None -> 0.1
- link left_wheel: mass None -> 0.5
- link right_wheel: mass None -> 0.5
- link sensor_mast: mass None -> 0.3

File: robots/rail_arm_robot.urdf (robot description, URDF)
Before this commit: robot rail_arm_robot, 6 links, 5 joints
Links:
- link elbow_link: mass None -> 0.3
- link end_effector: mass None -> 0.1
- link rail_platform_link: mass None -> 0.5
- link shoulder_link: mass None -> 0.5
- link world_link: mass None -> 5.0
- link wrist_link: mass None -> 0.2
