Commit message: fix: door_slide.urdf slide axis Y→X to match SDF convention
All rmf_demos SDF doors (clinic, hotel) define the prismatic slide
joint on local X axis (1 0 0).  The URDF had axis Y (0 1 0), so panels
slid perpendicular to the wall instead of along it.

File: robots/door_slide.urdf (robot description, URDF)
Before this commit: robot door_slide, 2 links, 1 joints
Joints:
- joint slide: axis 0 1 0 -> 1 0 0

Commit message: style: remove frame visual from door_slide.urdf
The frame link visual (gray pillar in center) was misleading for a
sliding door.  The fixed anchor point is invisible in practice
(embedded in wall).  Only the sliding panel needs a visual.

File: robots/door_slide.urdf (robot description, URDF)
Before this commit: robot door_slide, 2 links, 1 joints
Links:
- link frame: geometry 
